Commit message: -ing

File: moveit/isaac_moveit/config/panda.ros2_control.xacro (robot description, xacro)
@@ -1,5 +1,6 @@
 <?xml version="1.0"?>
 <robot xmlns:xacro="http://www.ros.org/wiki/xacro">
-    <xacro:macro name="panda_ros2_control" params="name initial_positions_file ros2_control_hardware_type">
+    <!-- <xacro:macro name="panda_ros2_control" params="name initial_positions_file ros2_control_hardware_type"> -->
+    <xacro:macro name="panda_ros2_control" params="name initial_positions_file ros2_control_hardware_type prefix:=''">
         <xacro:property name="initial_positions" value="${xacro.load_yaml(initial_positions_file)['initial_positions']}"/>
         <ros2_control name="${name}" type="system">
@@ -10,12 +11,13 @@
                 <xacro:if value="${ros2_control_hardware_type == 'isaac'}">
                     <plugin>topic_based_ros2_control/TopicBasedSystem</plugin>
-                    <param name="joint_commands_topic">/isaac_joint_commands</param>
-                    <param name="joint_states_topic">/isaac_joint_states</param>
+                    <param name="joint_commands_topic">/${prefix}isaac_joint_commands</param>
+                    <param name="joint_states_topic">/${prefix}isaac_joint_states</param>
                 </xacro:if>
             </hardware>
-            <joint name="panda_joint1">
+            <!-- <joint name="panda_joint1"> -->
+            <joint name="${prefix}panda_joint1">
                 <command_interface name="position"/>
                 <state_interface name="position">
-                  <param name="initial_value">${initial_positions['panda_joint1']}</param>
+                  <param name="initial_value">${initial_positions[prefix + 'panda_joint1']}</param>
                 </state_interface>
                 <state_interface name="velocity">
@@ -23,8 +25,9 @@
                 </state_interface>
             </joint>
-            <joint name="panda_joint2">
+            <!-- <joint name="panda_joint2"> -->
+            <joint name="${prefix}panda_joint2">
                 <command_interface name="position"/>
                 <state_interface name="position">
-                  <param name="initial_value">${initial_positions['panda_joint2']}</param>
+                  <param name="initial_value">${initial_positions[prefix + 'panda_joint2']}</param>
                 </state_interface>
                 <state_interface name="velocity">
@@ -32,8 +35,9 @@
                 </state_interface>
             </joint>
-            <joint name="panda_joint3">
+            <!-- <joint name="panda_joint3"> -->
+            <joint name="${prefix}panda_joint3">
                 <command_interface name="position"/>
                 <state_interface name="position">
-                  <param name="initial_value">${initial_positions['panda_joint3']}</param>
+                  <param name="initial_value">${initial_positions[prefix + 'panda_joint3']}</param>
                 </state_interface>
                 <state_interface name="velocity">
@@ -41,8 +45,9 @@
                 </state_interface>
             </joint>
-            <joint name="panda_joint4">
+            <!-- <joint name="panda_joint4"> -->
+            <joint name="${prefix}panda_joint4">
                 <command_interface name="position"/>
                 <state_interface name="position">
-                  <param name="initial_value">${initial_positions['panda_joint4']}</param>
+                  <param name="initial_value">${initial_positions[prefix + 'panda_joint4']}</param>
                 </state_interface>
                 <state_interface name="velocity">
@@ -50,8 +55,9 @@
                 </state_interface>
             </joint>
-            <joint name="panda_joint5">
+            <!-- <joint name="panda_joint5"> -->
+            <joint name="${prefix}panda_joint5">
                 <command_interface name="position"/>
                 <state_interface name="position">
-                  <param name="initial_value">${initial_positions['panda_joint5']}</param>
+                  <param name="initial_value">${initial_positions[prefix + 'panda_joint5']}</param>
                 </state_interface>
                 <state_interface name="velocity">
@@ -59,8 +65,9 @@
                 </state_interface>
             </joint>
-            <joint name="panda_joint6">
+            <!-- <joint name="panda_joint6"> -->
+            <joint name="${prefix}panda_joint6">
                 <command_interface name="position"/>
                 <state_interface name="position">
-                  <param name="initial_value">${initial_positions['panda_joint6']}</param>
+                  <param name="initial_value">${initial_positions[prefix + 'panda_joint6']}</param>
                 </state_interface>
                 <state_interface name="velocity">
@@ -68,8 +75,9 @@
                 </state_interface>
             </joint>
-            <joint name="panda_joint7">
+            <!-- <joint name="panda_joint7"> -->
+            <joint name="${prefix}panda_joint7">
                 <command_interface name="position"/>
                 <state_interface name="position">
-                  <param name="initial_value">${initial_positions['panda_joint7']}</param>
+                  <param name="initial_value">${initial_positions[prefix + 'panda_joint7']}</param>
                 </state_interface>
                 <state_interface name="velocity">

File: moveit/isaac_moveit/config/panda.urdf.xacro (robot description, xacro)
@@ -1,12 +1,18 @@
 <?xml version="1.0"?>
-<robot xmlns:xacro="http://www.ros.org/wiki/xacro" name="panda">
+<robot xmlns:xacro="http://www.ros.org/wiki/xacro" name="$(arg prefix)">
+    <xacro:arg name="prefix" default="" />
     <xacro:arg name="initial_positions_file" default="initial_positions.yaml" />
     <xacro:arg name="ros2_control_hardware_type" default="mock_components" />
-    <!-- Import panda urdf file -->
-    <xacro:include filename="$(find moveit_resources_panda_description)/urdf/panda.urdf" />
-    <!-- Import panda ros2_control description -->
+    <xacro:arg name="prefix" default="" /> <xacro:include filename="$(find isaac_moveit)/urdf/panda.urdf" />
     <xacro:include filename="panda.ros2_control.xacro" />
     <xacro:include filename="panda_hand.ros2_control.xacro" />
-    <xacro:panda_ros2_control name="PandaFakeSystem" initial_positions_file="$(arg initial_positions_file)" ros2_control_hardware_type="$(arg ros2_control_hardware_type)"/>
-    <xacro:panda_hand_ros2_control name="PandaHandFakeSystem" ros2_control_hardware_type="$(arg ros2_control_hardware_type)"/>
+    <xacro:panda_ros2_control
+        name="PandaFakeSystem"
+        initial_positions_file="$(arg initial_positions_file)"
+        ros2_control_hardware_type="$(arg ros2_control_hardware_type)"
+        prefix="$(arg prefix)" />
+    <xacro:panda_hand_ros2_control
+        name="PandaHandFakeSystem"
+        ros2_control_hardware_type="$(arg ros2_control_hardware_type)"
+        prefix="$(arg prefix)" />
 </robot>

File: moveit/isaac_moveit/config/panda_arm.xacro (robot description, xacro)
@@ -1,5 +1,6 @@
 <?xml version="1.0" ?>
 <robot xmlns:xacro="http://www.ros.org/wiki/xacro" name="panda">
-  <xacro:macro name="panda_arm">
+  <!-- <xacro:macro name="panda_arm"> -->
+    <xacro:macro name="panda_arm" params="prefix:=''">
     <!--GROUPS: Representation of a set of joints and links. This can be useful for specifying DOF to plan for, defining arms, end effectors, etc-->
     <!--LINKS: When a link is specified, the parent joint of that link (if it exists) is automatically included-->
@@ -8,57 +9,57 @@
     <!--SUBGROUPS: Groups can also be formed by referencing to already defined group names-->
     <group name="panda_arm">
-      <chain base_link="panda_link0" tip_link="panda_link8" />
+      <chain base_link="${prefix}/panda_link0" tip_link="${prefix}/panda_link8" />
     </group>
     <!--GROUP STATES: Purpose: Define a named state for a particular group, in terms of joint values. This is useful to define states like 'folded arms'-->
     <group_state name="ready" group="panda_arm">
-      <joint name="panda_joint1" value="0" />
-      <joint name="panda_joint2" value="-0.785" />
-      <joint name="panda_joint3" value="0" />
-      <joint name="panda_joint4" value="-2.356" />
-      <joint name="panda_joint5" value="0" />
-      <joint name="panda_joint6" value="1.571" />
-      <joint name="panda_joint7" value="0.785" />
+      <joint name="${prefix}/panda_joint1" value="0" />
+      <joint name="${prefix}/panda_joint2" value="-0.785" />
+      <joint name="${prefix}/panda_joint3" value="0" />
+      <joint name="${prefix}/panda_joint4" value="-2.356" />
+      <joint name="${prefix}/panda_joint5" value="0" />
+      <joint name="${prefix}/panda_joint6" value="1.571" />
+      <joint name="${prefix}/panda_joint7" value="0.785" />
     </group_state>
     <group_state name="extended" group="panda_arm">
-      <joint name="panda_joint1" value="0" />
-      <joint name="panda_joint2" value="0" />
-      <joint name="panda_joint3" value="0" />
-      <joint name="panda_joint4" value="0" />
-      <joint name="panda_joint5" value="0" />
-      <joint name="panda_joint6" value="1.571" />
-      <joint name="panda_joint7" value="0.785" />
+      <joint name="${prefix}/panda_joint1" value="0" />
+      <joint name="${prefix}/panda_joint2" value="0" />
+      <joint name="${prefix}/panda_joint3" value="0" />
+      <joint name="${prefix}/panda_joint4" value="0" />
+      <joint name="${prefix}/panda_joint5" value="0" />
+      <joint name="${prefix}/panda_joint6" value="1.571" />
+      <joint name="${prefix}/panda_joint7" value="0.785" />
     </group_state>
     <group_state name="transport" group="panda_arm">
-      <joint name="panda_joint1" value="0" />
-      <joint name="panda_joint2" value="-0.5599" />
-      <joint name="panda_joint3" value="0" />
-      <joint name="panda_joint4" value="-2.97" />
-      <joint name="panda_joint5" value="0" />
-      <joint name="panda_joint6" value="0" />
-      <joint name="panda_joint7" value="0.785" />
+      <joint name="${prefix}/panda_joint1" value="0" />
+      <joint name="${prefix}/panda_joint2" value="-0.5599" />
+      <joint name="${prefix}/panda_joint3" value="0" />
+      <joint name="${prefix}/panda_joint4" value="-2.97" />
+      <joint name="${prefix}/panda_joint5" value="0" />
+      <joint name="${prefix}/panda_joint6" value="0" />
+      <joint name="${prefix}/panda_joint7" value="0.785" />
     </group_state>
     <!--END EFFECTOR: Purpose: Represent information about an end effector.-->
     <!--VIRTUAL JOINT: Purpose: this element defines a virtual joint between a robot link and an external frame of reference (considered fixed with respect to the robot)-->
-    <virtual_joint name="virtual_joint" type="floating" parent_frame="world" child_link="panda_link0" />
+    <virtual_joint name="virtual_joint" type="floating" parent_frame="world" child_link="${prefix}/panda_link0" />
     <!--DISABLE COLLISIONS: By default it is assumed that any link of the robot could potentially come into collision with any other link in the robot. This tag disables collision checking between a specified pair of links. -->
-    <disable_collisions link1="panda_link0" link2="panda_link1" reason="Adjacent" />
-    <disable_collisions link1="panda_link0" link2="panda_link2" reason="Never" />
-    <disable_collisions link1="panda_link0" link2="panda_link3" reason="Never" />
-    <disable_collisions link1="panda_link0" link2="panda_link4" reason="Never" />
-    <disable_collisions link1="panda_link1" link2="panda_link2" reason="Adjacent" />
-    <disable_collisions link1="panda_link1" link2="panda_link3" reason="Never" />
-    <disable_collisions link1="panda_link1" link2="panda_link4" reason="Never" />
-    <disable_collisions link1="panda_link2" link2="panda_link3" reason="Adjacent" />
-    <disable_collisions link1="panda_link2" link2="panda_link4" reason="Never" />
-    <disable_collisions link1="panda_link2" link2="panda_link6" reason="Never" />
-    <disable_collisions link1="panda_link3" link2="panda_link4" reason="Adjacent" />
-    <disable_collisions link1="panda_link3" link2="panda_link5" reason="Never" />
-    <disable_collisions link1="panda_link3" link2="panda_link6" reason="Never" />
-    <disable_collisions link1="panda_link3" link2="panda_link7" reason="Never" />
-    <disable_collisions link1="panda_link4" link2="panda_link5" reason="Adjacent" />
-    <disable_collisions link1="panda_link4" link2="panda_link6" reason="Never" />
-    <disable_collisions link1="panda_link4" link2="panda_link7" reason="Never" />
-    <disable_collisions link1="panda_link5" link2="panda_link6" reason="Adjacent" />
-    <disable_collisions link1="panda_link6" link2="panda_link7" reason="Adjacent" />
+    <disable_collisions link1="${prefix}/panda_link0" link2="${prefix}/panda_link1" reason="Adjacent" />
+    <disable_collisions link1="${prefix}/panda_link0" link2="${prefix}/panda_link2" reason="Never" />
+    <disable_collisions link1="${prefix}/panda_link0" link2="${prefix}/panda_link3" reason="Never" />
+    <disable_collisions link1="${prefix}/panda_link0" link2="${prefix}/panda_link4" reason="Never" />
+    <disable_collisions link1="${prefix}/panda_link1" link2="${prefix}/panda_link2" reason="Adjacent" />
+    <disable_collisions link1="${prefix}/panda_link1" link2="${prefix}/panda_link3" reason="Never" />
+    <disable_collisions link1="${prefix}/panda_link1" link2="${prefix}/panda_link4" reason="Never" />
+    <disable_collisions link1="${prefix}/panda_link2" link2="${prefix}/panda_link3" reason="Adjacent" />
+    <disable_collisions link1="${prefix}/panda_link2" link2="${prefix}/panda_link4" reason="Never" />
+    <disable_collisions link1="${prefix}/panda_link2" link2="${prefix}/panda_link6" reason="Never" />
+    <disable_collisions link1="${prefix}/panda_link3" link2="${prefix}/panda_link4" reason="Adjacent" />
+    <disable_collisions link1="${prefix}/panda_link3" link2="${prefix}/panda_link5" reason="Never" />
+    <disable_collisions link1="${prefix}/panda_link3" link2="${prefix}/panda_link6" reason="Never" />
+    <disable_collisions link1="${prefix}/panda_link3" link2="${prefix}/panda_link7" reason="Never" />
+    <disable_collisions link1="${prefix}/panda_link4" link2="${prefix}/panda_link5" reason="Adjacent" />
+    <disable_collisions link1="${prefix}/panda_link4" link2="${prefix}/panda_link6" reason="Never" />
+    <disable_collisions link1="${prefix}/panda_link4" link2="${prefix}/panda_link7" reason="Never" />
+    <disable_collisions link1="${prefix}/panda_link5" link2="${prefix}/panda_link6" reason="Adjacent" />
+    <disable_collisions link1="${prefix}/panda_link6" link2="${prefix}/panda_link7" reason="Adjacent" />
   </xacro:macro>
 </robot>

File: moveit/isaac_moveit/config/panda_arm_hand.srdf.xacro (robot description, xacro)
@@ -4,9 +4,16 @@
     A URDF file must exist for this robot as well, where the joints and the links that are referenced are defined
 -->
-<robot xmlns:xacro="http://www.ros.org/wiki/xacro" name="panda">
+<!-- ttttttt -->
+<robot xmlns:xacro="http://www.ros.org/wiki/xacro" name="$(arg prefix)panda">
+  <xacro:arg name="prefix" default="franka_1_" />
+  <!-- ttttttt -->
   <xacro:include filename="$(find moveit_resources_panda_moveit_config)/config/panda_arm.xacro" />
   <xacro:include filename="$(find moveit_resources_panda_moveit_config)/config/hand.xacro" />
-  <xacro:panda_arm />
-  <xacro:hand />
+  <!-- ttttttt -->
+  <xacro:panda_arm prefix="$(arg prefix)"/>
+  <xacro:hand prefix="$(arg prefix)"/>
+  <!-- <xacro:panda_arm />
+  <xacro:hand /> -->
+  <!-- ttttttt -->
   <!--GROUPS: Representation of a set of joints and links. This can be useful for specifying DOF to plan for, defining arms, end effectors, etc-->
   <!--LINKS: When a link is specified, the parent joint of that link (if it exists) is automatically included-->
@@ -19,13 +26,22 @@
   </group>
   <group_state name="open" group="hand">
-    <joint name="panda_finger_joint1" value="0.035" />
-    <joint name="panda_finger_joint2" value="0.035" />
+  <!-- ttttttt -->
+    <!-- <joint name="panda_finger_joint1" value="0.035" />
+    <joint name="panda_finger_joint2" value="0.035" /> -->
+    <joint name="$(arg prefix)panda_finger_joint1" value="0.035" />
+    <joint name="$(arg prefix)panda_finger_joint2" value="0.035" />
+    <!-- ttttttt -->
   </group_state>
   <group_state name="close" group="hand">
-    <joint name="panda_finger_joint1" value="0" />
-    <joint name="panda_finger_joint2" value="0" />
+  <!-- ttttttt -->
+    <!-- <joint name="panda_finger_joint1" value="0" />
+    <joint name="panda_finger_joint2" value="0" /> -->
+    <joint name="$(arg prefix)panda_finger_joint1" value="0" />
+    <joint name="$(arg prefix)panda_finger_joint2" value="0" />
+    <!-- ttttttt -->
   </group_state>
   <!--END EFFECTOR: Purpose: Represent information about an end effector.-->
-  <end_effector name="hand" parent_link="panda_link8" group="hand" parent_group="panda_arm" />
+  <!-- <end_effector name="hand" parent_link="panda_link8" group="hand" parent_group="panda_arm" /> -->
+  <end_effector name="hand" parent_link="$(arg prefix)panda_link8" group="hand" parent_group="panda_arm" />
   <!--DISABLE COLLISIONS: By default it is assumed that any link of the robot could potentially come into collision with any other link in the robot. This tag disables collision checking between a specified pair of links. -->
   <disable_collisions link1="panda_hand" link2="panda_link3" reason="Never" />

File: moveit/isaac_moveit/config/panda_hand.ros2_control.xacro (robot description, xacro)
@@ -1,5 +1,6 @@
 <?xml version="1.0"?>
 <robot xmlns:xacro="http://www.ros.org/wiki/xacro">
-    <xacro:macro name="panda_hand_ros2_control" params="name ros2_control_hardware_type">
+    <!-- <xacro:macro name="panda_hand_ros2_control" params="name ros2_control_hardware_type"> -->
+    <xacro:macro name="panda_hand_ros2_control" params="name ros2_control_hardware_type prefix:=''">
         <ros2_control name="${name}" type="system">
             <hardware>
@@ -9,9 +10,12 @@
                 <xacro:if value="${ros2_control_hardware_type == 'isaac'}">
                     <plugin>topic_based_ros2_control/TopicBasedSystem</plugin>
-                    <param name="joint_commands_topic">/isaac_joint_commands</param>
-                    <param name="joint_states_topic">/isaac_joint_states</param>
+                    <!-- <param name="joint_commands_topic">/isaac_joint_commands</param>
+                    <param name="joint_states_topic">/isaac_joint_states</param> -->
+                    <param name="joint_commands_topic">/${prefix}isaac_joint_commands</param>
+                    <param name="joint_states_topic">/${prefix}isaac_joint_states</param>
                 </xacro:if>
             </hardware>
-            <joint name="panda_finger_joint1">
+            <!-- <joint name="panda_finger_joint1"> -->
+            <joint name="${prefix}panda_finger_joint1">
                 <command_interface name="position" />
                 <state_interface name="position">
@@ -22,6 +26,8 @@
                 </state_interface>
             </joint>
-            <joint name="panda_finger_joint2">
-                <param name="mimic">panda_finger_joint1</param>
+            <!-- <joint name="panda_finger_joint1"> -->
+            <joint name="${prefix}panda_finger_joint2">
+                <!-- <param name="mimic">panda_finger_joint1</param> -->
+                <param name="mimic">${prefix}panda_finger_joint1</param>
                 <param name="multiplier">1</param>
                 <command_interface name="position" />
